File: VCF.kicad_pcb (KiCad board)
At the start: 2 copper layers, 31 x 108 mm, 69 parts, among them J101 AudioJack2, J102 AudioJack2, J103 AudioJack2, J104 AudioJack2, J105 Conn_02x05_Odd_Even, J106 AudioJack2, Q101 2N3906, Q102 NST45010MW6T1G, Q103 2N3906, Q104 2N5457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

Commit message: fixed backwards cutoff frequency potentiometer
Connections:
- RV101 pad 1: +12V -> -12V
- RV101 pad 3: -12V -> +12V
Routing:
- net +12V: track 123.3 -> 130.2 mm, vias 7 -> 8
- net -12V: track 121.8 -> 120.9 mm, vias 0 -> 1
Other:
- board text added: "cutoff"
- board text added: "drive"
- board text added: "filter"
- board text added: "input"
- board text added: "ms-20 vcf version 2 chris defrancisci"
- board text added: "output"
- board text added: "resonance"
- board text removed: "ms-20 vcf version 1 chris defrancisci"
